File: Embedded_projects/PCB/ApiaryWaterDispensingSystem/_autosave-ApiaryWaterDispensingSystem.sch (KiCad schematic (older format))
At the start: 33 parts, among them J1 BME280, J10 Conn_02x19_Odd_Even, J11 DRV8835 PUMP, J12 PUMP, J13 BOOST, J14 POWER_5V, J15 SD CARD, J2 BH1750, J3 OLED, J4 RTC, J5 INA219 PV, J6 INA219 Battery, J7 Conn_02x19_Odd_Even, J8 I2C, J9 DRV8835 Control, SW1 SW_Push_Dual, SW2 SW_Push_Dual, SW3 SW_Push_Dual, SW4 SW_Push_Dual

Commit message: Update Kicad
+update eeschema
Parts:
- removed SW1, SW2, SW3, SW4: SW_Push_Dual, Button_Switch_THT:SW_PUSH-12mm, symbol Switch:SW_Push_Dual
- added J16: 3V3, Connector_PinSocket_2.54mm:PinSocket_1x02_P2.54mm_Vertical, symbol Connector:Conn_01x02_Female
- added SW1, SW2, SW3, SW4: SW_Push, Button_Switch_THT:SW_PUSH-12mm, symbol Switch:SW_Push
- J1, J5, J6: footprint (none) -> Connector_PinSocket_2.54mm:PinSocket_1x06_P2.54mm_Vertical
- J10, J7: footprint (none) -> Connector_PinSocket_2.54mm:PinSocket_2x20_P2.54mm_Vertical
- J2: footprint (none) -> Connector_PinSocket_2.54mm:PinSocket_1x05_P2.54mm_Vertical
- J3, J4: footprint (none) -> Connector_PinSocket_2.54mm:PinSocket_1x04_P2.54mm_Vertical
- J8: footprint (none) -> Connector_PinSocket_2.54mm:PinSocket_1x02_P2.54mm_Vertical
Connections:
- net +3V3: now also J3.2 (Pin_2), J16.1 (Pin_1); no longer J3.1 (Pin_1)
- net COUNTER_DOWN: now also J7.36 (Pin_36), SW2.2
- net COUNTER_UP: now also J7.38 (Pin_38), SW1.2
- net GND: now also J3.1 (Pin_1), J16.2 (Pin_2), SW1.1, SW2.1, SW3.1, SW4.1; no longer J3.2 (Pin_2), J5.2 (Pin_2)
- net OPTION: now also J7.34 (Pin_34), SW3.2
- net SPI3_MISO: now also J7.1 (Pin_1), J7.2 (Pin_2), J7.3 (Pin_3)
- net USER_ACTIVATED: now also J7.37 (Pin_37), SW4.2
Other:
- note added: "POWER SUPPLY"
- moved on the sheet: C1, C2, C3, C4, R10, R2, R4, R5, R6, R7, R8, R9
