File: Embedded_projects/PCB/ApiaryWaterDispensingSystem/ApiaryWaterDispensingSystem.sch (KiCad schematic (older format))
At the start: 33 parts, among them J1 BME280, J10 Conn_02x19_Odd_Even, J11 DRV8835 PUMP, J12 PUMP, J13 BOOST, J14 POWER_5V, J15 SD CARD, J2 BH1750, J3 OLED, J4 RTC, J5 INA219 PV, J6 INA219 Battery, J7 Conn_02x19_Odd_Even, J8 I2C, J9 DRV8835 Control, SW1 SW_Push_Dual, SW2 SW_Push_Dual, SW3 SW_Push_Dual, SW4 SW_Push_Dual

Commit message: +update project
positive test
Parts:
- removed J11: DRV8835 PUMP, symbol Connector:Conn_01x07_Female
- removed J9: DRV8835 Control, symbol Connector:Conn_01x07_Female
- removed SW1, SW2, SW3, SW4: SW_Push_Dual, Button_Switch_THT:SW_PUSH-12mm, symbol Switch:SW_Push_Dual
- added C10, C11, C12, C5, C6, C7, C8, C9: 100n, Capacitor_SMD:C_0805_2012Metric, symbol Device:C
- added J16: 3V3, Connector_PinSocket_2.54mm:PinSocket_1x02_P2.54mm_Vertical, symbol Connector:Conn_01x02_Female
- added J9: Conn_01x14_Male, ApiaryWaterDispensingSystem:PinSocket_1x07_P2.54mm_Vertical_DRV8835, symbol Connector:Conn_01x14_Male
- added SW1, SW2, SW3, SW4: SW_Push, Button_Switch_THT:SW_PUSH-12mm, symbol Switch:SW_Push
- C1, C2, C3, C4: footprint (none) -> Capacitor_SMD:C_0805_2012Metric
- J1: footprint (none) -> ApiaryWaterDispensingSystem:PinSocket_1x06_P2.54mm_Vertical_BME280
- J10, J7: footprint (none) -> Connector_PinSocket_2.54mm:PinSocket_2x19_P2.54mm_Vertical
- J12, J14: footprint Connector_PinHeader_2.54mm:PinHeader_1x02_P2.54mm_Vertical -> TerminalBlock_TE-Connectivity:TerminalBlock_TE_282834-2_1x02_P2.54mm_Horizontal
- J13: footprint Connector_PinHeader_2.54mm:PinHeader_1x03_P2.54mm_Vertical -> Connector_PinSocket_2.00mm:PinSocket_1x03_P2.00mm_Vertical
- J15: footprint (none) -> ApiaryWaterDispensingSystem:PinSocket_1x08_P2.54mm_Vertical_SD_CARD
- J2: footprint (none) -> Connector_PinSocket_2.54mm:PinSocket_1x05_P2.54mm_Vertical
- J3: footprint (none) -> Connector_PinSocket_2.54mm:PinSocket_1x04_P2.54mm_Vertical
- J4: footprint (none) -> ApiaryWaterDispensingSystem:PinSocket_1x04_P2.54mm_Vertical_RTCDS3231
- J5, J6: footprint (none) -> Connector_PinSocket_2.54mm:PinSocket_1x06_P2.54mm_Vertical
- J8: footprint (none) -> Connector_PinSocket_2.54mm:PinSocket_1x02_P2.54mm_Vertical
- R1, R3: value R -> 4k7
Connections:
- net +3V3: now also J3.2 (Pin_2), J4.2 (Pin_2), J7.16 (Pin_16), C10.2, C11.2, C12.2, C5.2, C6.1, C7.1, C8.1, C9.1, J16.1 (Pin_1), J9.2 (Pin_2); no longer J3.1 (Pin_1), J4.3 (Pin_3)
- net +6V: now also J9.9 (Pin_9)
- net AENABLE: now also J10.13 (Pin_13), J9.5 (Pin_5)
- net AOUT1: now also J9.13 (Pin_13); no longer J12.1 (Pin_1)
- net APHASE: now also J10.17 (Pin_17), J9.6 (Pin_6)
- net COUNTER_DOWN: now also J7.36 (Pin_36), SW2.2
- net COUNTER_UP: now also J7.38 (Pin_38), SW1.2
- net GND: now also J3.1 (Pin_1), J4.1 (Pin_1), J7.22 (Pin_22), C10.1, C11.1, C12.1, C5.1, C6.2, C7.2, C8.2, C9.2, J16.2 (Pin_2), J9.1 (Pin_1), SW1.1, SW2.1, SW3.1, SW4.1; no longer J3.2 (Pin_2), J4.4 (Pin_4)
- net GND1: now also J9.8 (Pin_8)
- net MODE: now also J10.15 (Pin_15), J9.7 (Pin_7)
- net OPTION: now also J7.34 (Pin_34), SW3.2
- net SCL: now also J4.4 (Pin_4); no longer J1.4 (Pin_4), J10.5 (Pin_5), J2.4 (Pin_4), J3.4 (Pin_4), J4.1 (Pin_1), J4.2 (Pin_2), J5.4 (Pin_4), J6.4 (Pin_4), J8.2 (Pin_2), R3.2
- net SPI3_MISO: now also J7.2 (Pin_2); no longer J15.4 (Pin_4), J15.5 (Pin_5)
- net USER_ACTIVATED: now also J7.37 (Pin_37), SW4.2
- net SPI3_SCK: now reaches J7.1 (Pin_1)
- net SPI3_SCK: now also J15.5 (Pin_5)
- net SPI3_MOSI: now reaches J7.3 (Pin_3)
- net SPI3_MOSI: now also J15.4 (Pin_4)
- net +BATT: no longer names the net of J7.33 (Pin_33)
- new net AOUT2: J12.1 (Pin_1), J9.12 (Pin_12)
- new net SDA: J1.4 (Pin_4), J10.5 (Pin_5), J2.4 (Pin_4), J3.4 (Pin_4), J4.3 (Pin_3), J5.4 (Pin_4), J6.4 (Pin_4), J8.2 (Pin_2), R3.2
- no-connect marks 12 -> 77
Other:
- note added: "MOTOR CONTROLLER"
- note added: "POWER SUPPLY"
- note added: "STM32 HEADER\n"
- note removed: "ARDUINO HEADER\n"
- note removed: "DRV8835 - Motor controller"
- moved on the sheet: C1, C2, C3, C4, J12, J13, J14, J15, R10, R2, R4, R5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
