File: Embedded_projects/PCB/Prototyp-ApiaryWDispensingSystem/PCB_ApiaryWaterDispensingSystem/MPPT.sch (KiCad schematic (older format))
At the start: 0 parts

Commit message: Many design changes have been added over the past few months #3
Parts:
- added U?: BQ76920PW, Package_SO:TSSOP-20_4.4x6.5mm_P0.65mm, symbol Battery_Management:BQ76920PW
Other:
- note added: "CELL Battery Monitor Family for Li-Ion"
- note added: "Solar managment for solar panel charging and step-down input"
Changed lines of the file:
@@
 $Descr A4 11693 8268
 encoding utf-8
-Sheet 3 9
+Sheet 3 10
 Title ""
 Date ""
@@
 Comment4 ""
 $EndDescr
+$Comp
+L Battery_Management:BQ76920PW U?
+U 1 1 68E2878D
+P 6275 2355
+F 0 "U?" H 6275 3336 50  0000 C CNN
+F 1 "BQ76920PW" H 6275 3245 50  0000 C CNN
+F 2 "Package_SO:TSSOP-20_4.4x6.5mm_P0.65mm" H 7175 1605 50  0001 C CNN
+F 3 "http://www.ti.com/lit/ds/symlink/bq76920.pdf" H 6975 2905 50  0001 C CNN
+	1    6275 2355
+	1    0    0    -1
+$EndComp
+Text Notes 5415 1155 0    50   ~ 0
+CELL Battery Monitor Family for Li-Ion
+Text Notes 1070 1185 0    50   ~ 0
+Solar managment for solar panel charging and step-down input
 $EndSCHEMATC
